Commit message: chui fort a ouai

File: urdf/heron_urdf.urdf (robot description, URDF)
Before this commit: robot heron, 9 links, 8 joints
Links:
- removed link custom
- link base_link: mass None -> 25
- link plate: mass None -> 0.389968906998643
- link support: mass None -> 0.389968906998643
- link wheel_bl: mass None -> 0.389968906998643
- link wheel_br: mass None -> 0.389968906998643
- link wheel_fl: mass None -> 0.389968906998643
- link wheel_fr: mass None -> 0.389968906998643
Joints:
- removed joint custom
